Commit message: add control

File: bumperbot_ws/install/bumperbot_description/share/bumperbot_description/urdf/bumperbot.gazebo.xacro (robot description, xacro)
@@ -1,4 +1,20 @@
 <?xml version="1.0"?>
 <robot xmlns:xacro="http://www.ros.org/wiki/xacro" name="bumperbot">
+    <transmission name="wheel_right_transmission">
+        <plugin>transmission_interface/simpleTransmission</plugin>
+        <joint name="right_wheel_joint" role="joint_right">
+            <mechanical_reduction>1</mechanical_reduction> <!-- 1:1 -->
+        </joint>
+        <actuator name="right_wheel_motor" role="actuator_right">
+        </actuator>
+    </transmission>
+    <transmission name="wheel_left_transmission">
+        <plugin>transmission_interface/simpleTransmission</plugin>
+        <joint name="left_wheel_joint" role="joint_left">
+            <mechanical_reduction>1</mechanical_reduction> <!-- 1:1 -->
+        </joint>
+        <actuator name="left_wheel_motor" role="actuator_left">
+        </actuator>
+    </transmission>
     <gazebo reference="left_wheel">
         <mu1>100000000000000.0</mu1>
@@ -35,3 +51,10 @@
         <maxVel>0.1</maxVel>
     </gazebo>
+    <gazebo>
+        <plugin filename="libgazebo_ros2_control.so" name="gazebo_ros2_control">
+            <robot_param>robot_description</robot_param> <!-- topic -->
+            <robot_param_node>robot_state_publisher</robot_param_node>
+            <parameters>$(find bumperbot_controller)/config/bumperbot_controllers.yaml</parameters>
+        </plugin>
+    </gazebo>
 </robot>

File: bumperbot_ws/install/bumperbot_description/share/bumperbot_description/urdf/bumperbot.urdf.xacro (robot description, xacro)
@@ -2,4 +2,5 @@
 <robot xmlns:xacro="http://www.ros.org/wiki/xacro" name="bumperbot">
 	<xacro:include filename="$(find bumperbot_description)/urdf/bumperbot.gazebo.xacro"/>
+	<xacro:include filename="$(find bumperbot_description)/urdf/bumperbot_ros2_control.xacro"/>
     <link name="base_footprint"/>
 	<!-- Base Link -->
